Commit message: add support for some crazyflie sensors

File: rotors_description/urdf/component_snippets.xacro (robot description, xacro)
@@ -831,4 +831,24 @@
     </xacro:imu_plugin_macro>
   </xacro:macro>
+  <xacro:macro name="mpu9250_smd_imu" params="namespace parent_link">
+    <!-- MPU-9250 SMD IMU. -->
+    <xacro:imu_plugin_macro
+      namespace="${namespace}"
+      imu_suffix=""
+      parent_link="${parent_link}"
+      imu_topic="imu"
+      mass_imu_sensor="0.00001"
+      gyroscope_noise_density="0.000175"
+      gyroscope_random_walk="0.0105"
+      gyroscope_bias_correlation_time="1000.0"
+      gyroscope_turn_on_bias_sigma="0.09"
+      accelerometer_noise_density="0.003"
+      accelerometer_random_walk="0.18"
+      accelerometer_bias_correlation_time="300.0"
+      accelerometer_turn_on_bias_sigma="0.588">
+      <inertia ixx="0.00001" ixy="0.0" ixz="0.0" iyy="0.00001" iyz="0.0" izz="0.00001" />
+      <origin xyz="0 0 0" rpy="0 0 0" />
+    </xacro:imu_plugin_macro>
+  </xacro:macro>
   <xacro:macro name="default_gps" params="namespace parent_link">
     <!-- Default GPS. -->
@@ -865,4 +885,21 @@
     </xacro:magnetometer_plugin_macro>
   </xacro:macro>
+  <xacro:macro name="mpu9250_smd_magnetometer" params="namespace parent_link">
+    <!-- MPU-9250 SMD Magnetometer. -->
+    <xacro:magnetometer_plugin_macro
+      namespace="${namespace}"
+      magnetometer_suffix=""
+      parent_link="${parent_link}"
+      magnetometer_topic="magnetic_field"
+      mass_magnetometer_sensor="0.00001"
+      ref_mag_north="0.000021493"
+      ref_mag_east="0.000000815"
+      ref_mag_down="0.000042795"
+      noise_normal="0.000000080 0.000000080 0.000000080"
+      noise_uniform_initial_bias="0.000000400 0.000000400 0.000000400">
+      <inertia ixx="0.00001" ixy="0.0" ixz="0.0" iyy="0.00001" iyz="0.0" izz="0.00001" />
+      <origin xyz="0 0 0" rpy="0 0 0" />
+    </xacro:magnetometer_plugin_macro>
+  </xacro:macro>
   <xacro:macro name="default_pressure_sensor" params="namespace parent_link">
     <xacro:pressure_sensor_plugin_macro
@@ -878,4 +915,20 @@
     </xacro:pressure_sensor_plugin_macro>
   </xacro:macro>
+  <xacro:macro name="lps25h_pressure_sensor" params="namespace parent_link">
+    <!-- LPS25H pressure sensor (TODO update params) -->
+    <xacro:pressure_sensor_plugin_macro
+      namespace="${namespace}"
+      pressure_sensor_suffix=""
+      parent_link="${parent_link}"
+      pressure_topic="air_pressure"
+      mass_pressure_sensor="0.00001"
+      reference_altitude="500.0"
+      pressure_variance="0.0">
+      <inertia ixx="0.00001" ixy="0.0" ixz="0.0" iyy="0.00001" iyz="0.0" izz="0.00001" />
+      <origin xyz="0 0 0" rpy="0 0 0" />
+    </xacro:pressure_sensor_plugin_macro>
+  </xacro:macro>
+  <!-- TODO add support of lps simulated sensor -->
+  <!--                                          -->
   <xacro:macro name="default_mavlink_interface" params="namespace imu_sub_topic rotor_count">
     <xacro:mavlink_interface_macro
